Commit message: Modify urdf and slam

File: description/lidar.xacro (robot description, xacro)
@@ -4,5 +4,5 @@
         <parent link="chassis"/>
         <child link="laser_frame"/>
-        <origin xyz="0.1 0 0.175" rpy="0 0 0"/>
+        <origin xyz="0.1 0 0.425" rpy="0 0 0"/>
     </joint>
     <link name="laser_frame">

File: description/robot_core.xacro (robot description, xacro)
@@ -36,18 +36,18 @@
     <link name="chassis">
         <visual>
-        <origin xyz="0.15 0 0.075"/>
+        <origin xyz="0.32 0 0.2"/>
             <geometry>
-                <box size="0.3 0.3 0.15"/>
+                <box size="0.64 0.64 0.4"/>
             </geometry>
             <material name="white"/>
         </visual>
         <collision>
-        <origin xyz="0.15 0 0.075"/>
+        <origin xyz="0.32 0 0.2"/>
             <geometry>
-                <box size="0.3 0.3 0.15"/>
+                <box size="0.64 0.64 0.4"/>
             </geometry>
         </collision>
-        <xacro:inertial_box mass="0.5" x="0.3" y="0.3" z="0.15">
-            <origin xyz="0.15 0 0.075" rpy="0 0 0"/>
+        <xacro:inertial_box mass="0.5" x="0.64" y="0.64" z="0.4">
+            <origin xyz="0.32 0 0.2" rpy="0 0 0"/>
         </xacro:inertial_box>
     </link>
